File: TestProj.kicad_pcb (KiCad board)
At the start: 2 copper layers, 0 parts

Commit message: early pcb routing
Parts:
- added C1: 0.1uF, Capacitor_SMD:C_0805_2012Metric, B.Cu at (110.4, 109.2)
- added C2: 0.1uF, Capacitor_SMD:C_0805_2012Metric, B.Cu at (103.5, 123.2)
- added C3: 22pF, Capacitor_SMD:C_0805_2012Metric, B.Cu at (110.4, 119.8)
- added C4: 22pF, Capacitor_SMD:C_0805_2012Metric, B.Cu at (110.4, 111.9)
- added C5: 0.1uF, Capacitor_SMD:C_0805_2012Metric, B.Cu at (93.2, 118.6)
- added C6: 10uF, Capacitor_SMD:C_0805_2012Metric, B.Cu at (93.2, 111.2)
- added C7: 1uF, Capacitor_SMD:C_0805_2012Metric, B.Cu at (103.2, 105.2)
- added D1: D_Small, Diode_SMD:D_SOD-123, B.Cu at (130.2, 98.5)
- added D2: D_Small, Diode_SMD:D_SOD-123, B.Cu at (130.2, 117.5)
- added D3: D_Small, Diode_SMD:D_SOD-123, B.Cu at (149.2, 98.5)
- added D4: D_Small, Diode_SMD:D_SOD-123, B.Cu at (149.2, 117.5)
- added F1: 500mA, Fuse:Fuse_1206_3216Metric, B.Cu at (91.4, 103.0)
- added MX1: MX-NoLED, MX_Only:MXOnly-1U, F.Cu at (122.2, 98.4)
- added MX2: MX-NoLED, MX_Only:MXOnly-1U, F.Cu at (122.2, 117.5)
- added MX3: MX-NoLED, MX_Only:MXOnly-1U, F.Cu at (141.3, 98.4)
- added MX4: MX-NoLED, MX_Only:MXOnly-1U, F.Cu at (141.3, 117.5)
- added R1: 22, Resistor_SMD:R_0805_2012Metric, B.Cu at (93.7, 102.4)
- added R2: 22, Resistor_SMD:R_0805_2012Metric, B.Cu at (95.9, 102.4)
- added R3: 10k, Resistor_SMD:R_0805_2012Metric, B.Cu at (108.1, 105.2)
- added R4: 10k, Resistor_SMD:R_0805_2012Metric, B.Cu at (99.8, 123.2)
- added SW1: SW_Push, random-keyboard-parts:SKQG-1155865, B.Cu at (105.3, 94.7)
- added U1: ATmega32U4-AU, Package_QFP:TQFP-44_10x10mm_P0.8mm, B.Cu at (101.6, 114.5)
- added USB1: Molex-0548190589, random-keyboard-parts:Molex-0548190589, B.Cu at (94.5, 90.8)
- added Y1: 16MHz, Crystal:Crystal_SMD_3225-4Pin_3.2x2.5mm, B.Cu at (110.5, 115.9)
Routing:
- net GND: track 0.00 -> 28.9 mm
- net +5V: track 0.00 -> 15.4 mm
- net Net-(C4-Pad1): track 0.00 -> 9.37 mm, vias 0 -> 2
- net Net-(R2-Pad1): track 0.00 -> 8.65 mm
- net Net-(R1-Pad1): track 0.00 -> 8.62 mm
- net Net-(C3-Pad1): track 0.00 -> 6.99 mm
- net VCC: track 0.00 -> 6.90 mm
- net D+: track 0.00 -> 6.81 mm
- net D-: track 0.00 -> 6.25 mm
- net Net-(C7-Pad1): track 0.00 -> 4.80 mm
Other:
- net class Default: trace_width 0.25 -> 0.254
- net class Power added: clearance 0.2, trace_width 0.381, via_dia 0.8, via_drill 0.4
